Commit message: Restored proper rviz launch file with interactive markers

File: config/srdf/tiago.srdf.xacro (robot description, xacro)
@@ -4,27 +4,36 @@
     A URDF file must exist for this robot as well, where the joints and the links that are referenced are defined
 -->
-<robot name="tiago" xmlns:xacro="http://ros.org/wiki/xacro">
+<robot xmlns:xacro="http://ros.org/wiki/xacro" name="tiago">
+    <!-- ARGUMENTS -->
+    <!-- pmb2, omni_base -->
     <xacro:arg name="base_type" default="pmb2"/>
-    <xacro:arg name="arm_model" default="tiago-arm"/>
-    <xacro:arg name="end_effector" default="pal-hey5"/>
+    <!-- no-arm, tiago-arm -->
+    <xacro:arg name="arm_type" default="tiago-arm"/>
+    <!-- no-ft-sensor, schunk-ft -->
     <xacro:arg name="ft_sensor" default="schunk-ft"/>
+    <!-- no-end-effector, pal-gripper, pal-hey5, custom, robotiq-2f-85,robotiq-2f-140-->
+    <xacro:arg name="end_effector" default="pal-gripper"/>
+    <!-- PROPERTIES -->
+    <!-- HW configuration -->
     <xacro:property name="base_type" value="$(arg base_type)"/>
-    <xacro:property name="arm_model" value="$(arg arm_model)"/>
-    <xacro:property name="has_arm" value="${arm_model not in ['no-arm']}"/>
+    <xacro:property name="arm_type" value="$(arg arm_type)"/>
     <xacro:property name="end_effector" value="$(arg end_effector)"/>
     <xacro:property name="ft_sensor" value="$(arg ft_sensor)"/>
-    <xacro:property name="has_ft_sensor" value="${ft_sensor not in ['no-ft-sensor']}"/>
+    <!-- HW configuration helpers-->
+    <xacro:property name="has_ft_sensor" value="${ft_sensor != 'no-ft-sensor'}"/>
     <xacro:property name="robot" value="tiago"/>
-    <xacro:property name="end_effector_arg" value="$(arg end_effector)"/>
-<!-- <virtual_joint name="odom_to_base" child_link="base_footprint" parent_frame="odom" type="planar"/> -->
-<xacro:if value="${base_type == 'omni_base'}">
-    <xacro:property name="robot" value="tiago_omni"/>
-</xacro:if>
-<xacro:unless value="${base_type == 'omni_base'}">
-    <xacro:property name="robot" value="tiago"/>
-</xacro:unless>
-<xacro:if value="${end_effector == 'no-end-effector'}">
-    <xacro:property name="end_effector_arg" value="no-ee"/>
-</xacro:if>
+    <xacro:property name="has_arm" value="${arm_type != 'no-arm'}"/>
+    <!-- This arg is needed to pass no-ee instead of no-end-effector -->
+    <xacro:property name="end_effector_arg" value="${end_effector}"/>
+    <xacro:if value="${end_effector_arg == 'no-end-effector'}">
+        <xacro:property name="end_effector_arg" value="no-ee"/>
+    </xacro:if>
+    <!-- HW configuration check -->
+    <xacro:if value="${base_type == 'omni_base'}">
+        <xacro:property name="robot" value="tiago_omni"/>
+    </xacro:if>
+    <xacro:unless value="${base_type == 'omni_base'}">
+        <xacro:property name="robot" value="tiago"/>
+    </xacro:unless>
     <!--GROUPS: Representation of a set of joints and links. This can be useful for specifying DOF to plan for, defining arms, end effectors, etc-->
     <!--LINKS: When a link is specified, the parent joint of that link (if it exists) is automatically included-->
@@ -32,40 +41,43 @@
     <!--CHAINS: When a chain is specified, all the links along the chain (including endpoints) are included in the group. Additionally, all the joints that are parents to included links are also included. This means that joints along the chain and the parent joint of the base link are included in the group-->
     <!--SUBGROUPS: Groups can also be formed by referencing to already defined group names-->
-<xacro:if value="${has_arm}">
-    <group name="arm">
-        <joint name="arm_1_joint" />
-        <joint name="arm_2_joint" />
-        <joint name="arm_3_joint" />
-        <joint name="arm_4_joint" />
-        <joint name="arm_5_joint" />
-        <joint name="arm_6_joint" />
-        <joint name="arm_7_joint" />
-        <joint name="arm_tool_joint" />
-    </group>
-    <group name="arm_torso">
-        <joint name="torso_lift_joint" />
-        <joint name="arm_1_joint" />
-        <joint name="arm_2_joint" />
-        <joint name="arm_3_joint" />
-        <joint name="arm_4_joint" />
-        <joint name="arm_5_joint" />
-        <joint name="arm_6_joint" />
-        <joint name="arm_7_joint" />
-        <joint name="arm_tool_joint" />
-    </group>
-    <xacro:include filename="$(find tiago_moveit_config)/config/srdf/end_effectors/${end_effector}.srdf.xacro" />
-    <xacro:define_end_effector arm="arm" name="${end_effector_name}"/>
-    <xacro:if value="${has_ft_sensor}">
-        <xacro:include filename="$(find tiago_moveit_config)/config/srdf/disable_collisions/${robot}_${end_effector_arg}_${ft_sensor}.srdf.xacro" />
+    <xacro:if value="${has_arm}">
+        <!-- Arm group -->
+        <group name="arm">
+            <joint name="arm_1_joint" />
+            <joint name="arm_2_joint" />
+            <joint name="arm_3_joint" />
+            <joint name="arm_4_joint" />
+            <joint name="arm_5_joint" />
+            <joint name="arm_6_joint" />
+            <joint name="arm_7_joint" />
+            <joint name="arm_tool_joint" />
+        </group>
+        <!-- Arm with torso group -->
+        <group name="arm_torso">
+            <joint name="torso_lift_joint" />
+            <joint name="arm_1_joint" />
+            <joint name="arm_2_joint" />
+            <joint name="arm_3_joint" />
+            <joint name="arm_4_joint" />
+            <joint name="arm_5_joint" />
+            <joint name="arm_6_joint" />
+            <joint name="arm_7_joint" />
+            <joint name="arm_tool_joint" />
+        </group>
+        <xacro:include filename="$(find tiago_moveit_config)/config/srdf/end_effectors/${end_effector}.srdf.xacro" />
+        <xacro:define_end_effector arm="arm" name="${end_effector_name}"/>
+        <xacro:if value="${has_ft_sensor}">
+            <xacro:include filename="$(find tiago_moveit_config)/config/srdf/disable_collisions/${robot}_${end_effector_arg}_${ft_sensor}.srdf.xacro" />
+        </xacro:if>
+        <xacro:unless value="${has_ft_sensor}">
+            <xacro:include filename="$(find tiago_moveit_config)/config/srdf/disable_collisions/${robot}_${end_effector_arg}.srdf.xacro" />
+        </xacro:unless>
     </xacro:if>
-    <xacro:unless value="${has_ft_sensor}">
-        <xacro:include filename="$(find tiago_moveit_config)/config/srdf/disable_collisions/${robot}_${end_effector_arg}.srdf.xacro" />
+    <xacro:unless value="${has_arm}">
+        <!-- Just torso group -->
+        <group name="torso">
+            <joint name="torso_lift_joint" />
+        </group>
+        <xacro:include filename="$(find tiago_moveit_config)/config/srdf/disable_collisions/${robot}_no-arm.srdf.xacro" />
     </xacro:unless>
-</xacro:if>
-<xacro:unless value="${has_arm}">
-    <group name="torso">
-        <joint name="torso_lift_joint" />
-    </group>
-    <xacro:include filename="$(find tiago_moveit_config)/config/srdf/disable_collisions/${robot}_no-arm.srdf.xacro" />
-</xacro:unless>
 </robot>
